Commit message: slitely modify of urdf and train

File: loco_manipulation_gym/resources/robots/XbT/urdf/XbT.urdf (robot description, URDF)
Before this commit: robot XbT, 10 links, 9 joints
Links:
- link left_calf_Link: geometry collision box size=0.15 0.01 0.06; visual mesh filename=../meshes/left_calf_Link.STL
- link right_calf_Link: geometry collision box size=0.15 0.01 0.06; visual mesh filename=../meshes/right_calf_Link.STL
Joints:
- joint left_calf: limit lower=-3.14 upper=3.14 effort=35 velocity=25 -> lower=-1.0 upper=0.42 effort=35 velocity=25
- joint left_leg: limit lower=-3.14 upper=3.14 effort=35 velocity=25 -> lower=-0.5 upper=1.5 effort=35 velocity=25
- joint left_thigh: limit lower=-3.14 upper=3.14 effort=35 velocity=25 -> lower=-1.2 upper=0.7 effort=35 velocity=25
- joint right_calf: limit lower=-3.14 upper=3.14 effort=35 velocity=25 -> lower=-0.42 upper=1.0 effort=35 velocity=25
- joint right_leg: limit lower=-3.14 upper=3.14 effort=35 velocity=25 -> lower=-1.5 upper=0.5 effort=35 velocity=25
- joint right_thigh: limit lower=-3.14 upper=3.14 effort=35 velocity=25 -> lower=-0.7 upper=1.2 effort=35 velocity=25
